File: led_watch_v1.sch (KiCad schematic (older format))
At the start: 0 parts

Commit message: Pulled new library updates
Changed lines of the file:
@@
 LIBS:connex_Resistor
 LIBS:connex_test
+LIBS:led_watch_v1-cache
 EELAYER 25 0
 EELAYER END
@@
 $EndDescr
 $Sheet
-S 1825 2150 1850 1600
+S 1625 1400 1850 1600
 U 5A2D4EF8
 F0 "leds" 60
