File: leds.sch (KiCad schematic (older format))
At the start: 27 parts

Commit message: Pulled new library updates
Parts:
- added C? (x3): CONNEX-SMD-CAP-10UF-0402, Capacitors_SMD:C_0402, symbol CONNEX-SMD-CAP-10UF-0402
Changed lines of the file:
@@
 LIBS:connex_Resistor
 LIBS:connex_test
+LIBS:led_watch_v1-cache
 EELAYER 25 0
 EELAYER END
@@
 Text Label 2400 6775 0    60   ~ 0
 LED_AGREEN
+$Comp
+L CONNEX-SMD-CAP-10UF-0402 C?
+U 1 1 5A2DD3DF
+P 9100 3450
+F 0 "C?" H 9110 3520 50  0000 L CNN
+F 1 "CONNEX-SMD-CAP-10UF-0402" H 8850 3975 20  0001 L CNN
+F 2 "Capacitors_SMD:C_0402" H 9100 3625 20  0001 C CNN
+F 3 "N/A" H 9100 3675 20  0001 C CNN
+F 4 "81-GRJ155R60J106ME1D" H 9100 3775 20  0001 C CNN "SUPPLIER PART"
+F 5 "MOUSER" H 9100 3825 20  0001 C CNN "SUPPLIER"
+F 6 "GRJ155R60J106ME11D" H 9100 3875 20  0001 C CNN "MPN"
+F 7 "https://www.mouser.com/ProductDetail/Murata-Electronics/GRJ155R60J106ME11D/?qs=sGAEpiMZZMs0AnBnWHyRQO9VYadaKTO%252b4wiupwT68VQ9yfSZ%252bJ8BuA%3d%3d" H 9100 3725 20  0001 C CNN "LINK"
+F 8 "SAMSUNG ELECTRO-MECHANICS" H 9100 3925 20  0001 C CNN "MANUFACTURER"
+F 9 "YES" H 9050 3525 20  0001 C CNN "PLACE"
+F 10 "10UF" H 9200 3375 40  0000 C CNN "CAPACITANCE"
+F 11 "6.3V" H 9200 3325 40  0001 C CNN "VOLTAGE"
+	1    9100 3450
+	1    0    0    -1
+$EndComp
+$Comp
+L CONNEX-SMD-CAP-10UF-0402 C?
+U 1 1 5A2DD598
+P 9300 3850
+F 0 "C?" H 9310 3920 50  0000 L CNN
+F 1 "CONNEX-SMD-CAP-10UF-0402" H 9050 4375 20  0001 L CNN
+F 2 "Capacitors_SMD:C_0402" H 9300 4025 20  0001 C CNN
+F 3 "N/A" H 9300 4075 20  0001 C CNN
+F 4 "81-GRJ155R60J106ME1D" H 9300 4175 20  0001 C CNN "SUPPLIER PART"
+F 5 "MOUSER" H 9300 4225 20  0001 C CNN "SUPPLIER"
+F 6 "GRJ155R60J106ME11D" H 9300 4275 20  0001 C CNN "MPN"
+F 7 "https://www.mouser.com/ProductDetail/Murata-Electronics/GRJ155R60J106ME11D/?qs=sGAEpiMZZMs0AnBnWHyRQO9VYadaKTO%252b4wiupwT68VQ9yfSZ%252bJ8BuA%3d%3d" H 9300 4125 20  0001 C CNN "LINK"
+F 8 "SAMSUNG ELECTRO-MECHANICS" H 9300 4325 20  0001 C CNN "MANUFACTURER"
+F 9 "YES" H 9250 3925 20  0001 C CNN "PLACE"
+F 10 "10UF" H 9400 3775 40  0000 C CNN "CAPACITANCE"
+F 11 "6.3V" H 9400 3725 40  0001 C CNN "VOLTAGE"
+	1    9300 3850
+	1    0    0    -1
+$EndComp
+$Comp
+L CONNEX-SMD-CAP-10UF-0402 C?
+U 1 1 5A2DD659
+P 9300 4400
+F 0 "C?" H 9310 4470 50  0000 L CNN
+F 1 "CONNEX-SMD-CAP-10UF-0402" H 9050 4925 20  0001 L CNN
+F 2 "Capacitors_SMD:C_0402" H 9300 4575 20  0001 C CNN
+F 3 "N/A" H 9300 4625 20  0001 C CNN
+F 4 "81-GRJ155R60J106ME1D" H 9300 4725 20  0001 C CNN "SUPPLIER PART"
+F 5 "MOUSER" H 9300 4775 20  0001 C CNN "SUPPLIER"
+F 6 "GRJ155R60J106ME11D" H 9300 4825 20  0001 C CNN "MPN"
+F 7 "https://www.mouser.com/ProductDetail/Murata-Electronics/GRJ155R60J106ME11D/?qs=sGAEpiMZZMs0AnBnWHyRQO9VYadaKTO%252b4wiupwT68VQ9yfSZ%252bJ8BuA%3d%3d" H 9300 4675 20  0001 C CNN "LINK"
+F 8 "SAMSUNG ELECTRO-MECHANICS" H 9300 4875 20  0001 C CNN "MANUFACTURER"
+F 9 "YES" H 9250 4475 20  0001 C CNN "PLACE"
+F 10 "10UF" H 9400 4325 40  0000 C CNN "CAPACITANCE"
+F 11 "6.3V" H 9400 4275 40  0001 C CNN "VOLTAGE"
+	1    9300 4400
+	1    0    0    -1
+$EndComp
 $EndSCHEMATC
